File: QS-13u.kicad_sch (KiCad schematic)
At the start: 98 parts, among them J1 Conn_01x04, J2 USB_C_Receptacle_USB2.0, SW1 MX_SW_solder, SW10 MX_SW_solder, SW11 MX_SW_solder, SW12 MX_SW_solder, SW13 MX_SW_solder, SW14 MX_SW_solder, SW15 MX_SW_solder, SW16 MX_SW_solder, SW17 MX_SW_solder, SW18 MX_SW_solder, SW19 MX_SW_solder, SW2 MX_SW_solder, SW20 MX_SW_solder, SW21 MX_SW_solder, SW22 MX_SW_solder, SW23 MX_SW_solder, SW24 MX_SW_solder, SW25 MX_SW_solder, SW26 MX_SW_solder, SW27 MX_SW_solder, SW28 MX_SW_solder, SW29 MX_SW_solder, SW3 MX_SW_solder, SW30 MX_SW_solder, SW31 MX_SW_solder, SW32 MX_SW_solder, SW33 MX_SW_solder, SW34 MX_SW_solder, SW35 MX_SW_solder, SW36 MX_SW_solder, SW37 MX_SW_solder, SW38 MX_SW_solder, SW39 MX_SW_solder, SW4 MX_SW_solder, SW40 MX_SW_solder, SW41 MX_SW_solder, SW42 MX_SW_solder, SW43 MX_SW_solder, SW44 MX_SW_solder, SW45 MX_SW_solder, SW46 MX_SW_solder, SW47 MX_SW_solder, SW48 MX_SW_solder, SW49 MX_SW_solder, SW5 MX_SW_solder, SW50 MX_SW_solder, SW51 SW_Push, SW6 MX_SW_solder, SW7 MX_SW_solder, SW8 MX_SW_solder, SW9 MX_SW_solder, U1 USBLC6-2SC6, U2 ATmega32U2-M, Y1 16 MHz

Commit message: Undocumented progress
Parts:
- gave numbers to parts that had none: 4
- renumbered SW48 to SW50, SW49 to SW51, SW50 to SW54, SW51 to SW55
Changed lines of the file:
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@@
   (symbol (lib_id "marbastlib-mx:MX_SW_solder") (at 83.82 71.374 0) (unit 1)
     (in_bom yes) (on_board yes)
-    (property "Reference" "SW48" (id 0) (at 83.82 67.056 0))
+    (property "Reference" "SW50" (id 0) (at 83.82 67.056 0))
     (property "Value" "MX_SW_solder" (id 1) (at 83.82 66.294 0)
       (effects (font (size 1.27 1.27)) hide)
@@
   (symbol (lib_id "marbastlib-mx:MX_SW_solder") (at 25.4 71.374 0) (unit 1)
     (in_bom yes) (on_board yes)
-    (property "Reference" "SW?" (id 0) (at 25.4 67.056 0))
+    (property "Reference" "SW48" (id 0) (at 25.4 67.056 0))
     (property "Value" "MX_SW_solder" (id 1) (at 25.4 66.294 0)
       (effects (font (size 1.27 1.27)) hide)
@@
   (symbol (lib_id "marbastlib-mx:MX_SW_solder") (at 171.45 71.374 0) (unit 1)
     (in_bom yes) (on_board yes)
-    (property "Reference" "SW?" (id 0) (at 171.45 67.056 0))
+    (property "Reference" "SW53" (id 0) (at 171.45 67.056 0))
     (property "Value" "MX_SW_solder" (id 1) (at 171.45 66.294 0)
       (effects (font (size 1.27 1.27)) hide)
@@
   (symbol (lib_id "marbastlib-mx:MX_SW_solder") (at 54.61 71.374 0) (unit 1)
     (in_bom yes) (on_board yes)
-    (property "Reference" "SW?" (id 0) (at 54.61 67.056 0))
+    (property "Reference" "SW49" (id 0) (at 54.61 67.056 0))
     (property "Value" "MX_SW_solder" (id 1) (at 54.61 66.294 0)
       (effects (font (size 1.27 1.27)) hide)
@@
   (symbol (lib_id "marbastlib-mx:MX_SW_solder") (at 104.14 71.374 90) (unit 1)
     (in_bom yes) (on_board yes)
-    (property "Reference" "SW49" (id 0) (at 102.362 67.31 90)
+    (property "Reference" "SW51" (id 0) (at 102.362 67.31 90)
       (effects (font (size 1.27 1.27)) (justify right))
     )
@@
   (symbol (lib_id "marbastlib-mx:MX_SW_solder") (at 191.77 71.374 90) (unit 1)
     (in_bom yes) (on_board yes)
-    (property "Reference" "SW50" (id 0) (at 189.738 74.422 90)
+    (property "Reference" "SW54" (id 0) (at 189.738 74.422 90)
       (effects (font (size 1.27 1.27)) (justify right))
     )
@@
   (symbol (lib_id "marbastlib-mx:MX_SW_solder") (at 142.24 71.374 0) (unit 1)
     (in_bom yes) (on_board yes)
-    (property "Reference" "SW?" (id 0) (at 142.24 67.056 0))
+    (property "Reference" "SW52" (id 0) (at 142.24 67.056 0))
     (property "Value" "MX_SW_solder" (id 1) (at 142.24 66.294 0)
       (effects (font (size 1.27 1.27)) hide)
@@
   (symbol (lib_id "Switch:SW_Push") (at 48.514 106.172 0) (unit 1)
     (in_bom yes) (on_board yes) (fields_autoplaced)
-    (property "Reference" "SW51" (id 0) (at 48.514 98.552 0))
+    (property "Reference" "SW55" (id 0) (at 48.514 98.552 0))
     (property "Value" "SW_Push" (id 1) (at 48.514 101.092 0))
     (property "Footprint" "Button_Switch_SMD:SW_SPST_SKQG_WithStem" (id 2) (at 48.514 101.092 0)
@@
       (reference "SW47") (unit 1) (value "MX_SW_solder") (footprint "marbastlib-mx:SW_MX_1u")
     )
+    (path "/0f1c5d63-1d32-4ff6-8d93-dcf5c1c03c03"
+      (reference "SW48") (unit 1) (value "MX_SW_solder") (footprint "marbastlib-mx:SW_MX_1.5u")
+    )
+    (path "/5a904dcc-2f93-4281-8e8f-655976fc8404"
+      (reference "SW49") (unit 1) (value "MX_SW_solder") (footprint "marbastlib-mx:SW_MX_1.5u")
+    )
     (path "/0b5753cc-f737-4e82-b31f-7809688696d9"
-      (reference "SW48") (unit 1) (value "MX_SW_solder") (footprint "marbastlib-mx:SW_MX_1u")
+      (reference "SW50") (unit 1) (value "MX_SW_solder") (footprint "marbastlib-mx:SW_MX_1u")
     )
     (path "/89a1b2f6-56a0-4e43-9426-28b8440b4c1b"
-      (reference "SW49") (unit 1) (value "MX_SW_solder") (footprint "marbastlib-mx:SW_MX_1u")
+      (reference "SW51") (unit 1) (value "MX_SW_solder") (footprint "marbastlib-mx:SW_MX_1u")
+    )
+    (path "/c02ba2ca-342f-41cf-80ff-4493cff37acc"
+      (reference "SW52") (unit 1) (value "MX_SW_solder") (footprint "marbastlib-mx:SW_MX_1.5u")
+    )
+    (path "/2e01b078-f7ca-4c89-986c-02a4a28501e2"
+      (reference "SW53") (unit 1) (value "MX_SW_solder") (footprint "marbastlib-mx:SW_MX_1.5u")
     )
     (path "/b18cbbf2-93ad-4294-9a17-d9e43ca0d7be"
-      (reference "SW50") (unit 1) (value "MX_SW_solder") (footprint "marbastlib-mx:SW_MX_1.25u")
+      (reference "SW54") (unit 1) (value "MX_SW_solder") (footprint "marbastlib-mx:SW_MX_1.25u")
     )
     (path "/d27f2b02-a3d0-4a4e-9163-dbab4452129c"
-      (reference "SW51") (unit 1) (value "SW_Push") (footprint "Button_Switch_SMD:SW_SPST_SKQG_WithStem")
-    )
-    (path "/0f1c5d63-1d32-4ff6-8d93-dcf5c1c03c03"
-      (reference "SW?") (unit 1) (value "MX_SW_solder") (footprint "marbastlib-mx:SW_MX_1.5u")
-    )
-    (path "/2e01b078-f7ca-4c89-986c-02a4a28501e2"
-      (reference "SW?") (unit 1) (value "MX_SW_solder") (footprint "marbastlib-mx:SW_MX_1.5u")
-    )
-    (path "/5a904dcc-2f93-4281-8e8f-655976fc8404"
-      (reference "SW?") (unit 1) (value "MX_SW_solder") (footprint "marbastlib-mx:SW_MX_1.5u")
-    )
-    (path "/c02ba2ca-342f-41cf-80ff-4493cff37acc"
-      (reference "SW?") (unit 1) (value "MX_SW_solder") (footprint "marbastlib-mx:SW_MX_1.5u")
+      (reference "SW55") (unit 1) (value "SW_Push") (footprint "Button_Switch_SMD:SW_SPST_SKQG_WithStem")
     )
     (path "/e0f9fec8-73fa-41e1-949f-b3b3870bdbd3"
