File: pcb/QS-13u.kicad_pcb (KiCad board)
At the start: 2 copper layers, 247.7 x 84.9 mm, 98 parts, among them J1 Conn_01x04, J2 USB_C_Receptacle_USB2.0, SW1 MX_SW_solder, SW10 MX_SW_solder, SW11 MX_SW_solder, SW12 MX_SW_solder, SW13 MX_SW_solder, SW14 MX_SW_solder, SW15 MX_SW_solder, SW16 MX_SW_solder, SW17 MX_SW_solder, SW18 MX_SW_solder, SW19 MX_SW_solder, SW2 MX_SW_solder, SW20 MX_SW_solder, SW21 MX_SW_solder, SW22 MX_SW_solder, SW23 MX_SW_solder, SW24 MX_SW_solder, SW25 MX_SW_solder, SW26 MX_SW_solder, SW27 MX_SW_solder, SW28 MX_SW_solder, SW29 MX_SW_solder, SW3 MX_SW_solder, SW30 MX_SW_solder, SW31 MX_SW_solder, SW32 MX_SW_solder, SW33 MX_SW_solder, SW34 MX_SW_solder, SW35 MX_SW_solder, SW36 MX_SW_solder, SW37 MX_SW_solder, SW38 MX_SW_solder, SW39 MX_SW_solder, SW4 MX_SW_solder, SW40 MX_SW_solder, SW41 MX_SW_solder, SW42 MX_SW_solder, SW43 MX_SW_solder, SW44 MX_SW_solder, SW45 MX_SW_solder, SW46 MX_SW_solder, SW47 MX_SW_solder, SW48 MX_SW_solder, SW49 MX_SW_solder, SW5 MX_SW_solder, SW50 MX_SW_solder, SW51 MX_SW_solder, SW52 MX_SW_solder, SW53 MX_SW_solder, SW54 MX_SW_solder, SW55 SW_Push, SW6 MX_SW_solder, SW7 MX_SW_solder, SW8 MX_SW_solder, SW9 MX_SW_solder, U1 USBLC6-2SC6, U2 ATmega32U2-M, Y1 16 MHz

Commit message: Fixes + Updates
- Fixed some weird submodules shenanigans
- Repositioned the JST connector
- Adjusted the outline for gummy o-ring mount
Parts:
- added R4: 10k, Resistor_SMD:R_0603_1608Metric, B.Cu at (55.9, 56.7)
- added R5: 10k, Resistor_SMD:R_0603_1608Metric, B.Cu at (57.5, 56.7)
- moved U1 60.3 mm to (71.4, 50.8), turned to 0 degrees
- moved J1 55.8 mm to (80.3, 50.8), turned to -90 degrees
- moved R6 37.4 mm to (63.1, 74.4), turned to -45 degrees
- moved C1 29.5 mm to (64.5, 68.5), turned to 45 degrees
- moved U2 28.8 mm to (59.9, 70.9), turned to -135 degrees
- moved D17 25.8 mm to (217.5, 81.8)
- moved S6 25.8 mm to (260.4, 41.3)
- moved SW13 25.8 mm to (260.4, 41.3)
- moved D20 25.8 mm to (96.0, 100.8)
- moved F1 25.8 mm to (142.1, 45.2)
- moved SW1 25.8 mm to (41.3, 41.3)
- moved SW2 25.8 mm to (60.3, 41.3)
- moved SW29 25.8 mm to (112.7, 79.4)
- moved D1 25.8 mm to (50.8, 43.7)
- moved D14 25.8 mm to (103.2, 81.8)
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- renumbered R4 to R6
Connections:
- U2 pad 29: D+ -> Net-(R4-Pad2)
- U2 pad 30: D- -> Net-(R5-Pad1)
Routing:
- net D+: track 0.00 -> 16.8 mm
- net D-: track 0.00 -> 15.5 mm
- net Net-(R4-Pad2): track 0.00 -> 12.5 mm
- net Net-(R5-Pad1): track 0.00 -> 12.0 mm
- net GND: track 0.00 -> 11.8 mm
- net UD+: track 0.00 -> 5.93 mm
- net UD-: track 0.00 -> 5.93 mm
- net +5V: track 0.00 -> 5.87 mm
- net Net-(U2-Pad1): track 0.00 -> 3.30 mm
- net Net-(U2-Pad2): track 0.00 -> 3.24 mm
- net Net-(C3-Pad1): track 0.00 -> 2.43 mm
Other:
- board size 247.7 x 84.9 mm -> 247.6 x 84.9 mm

Commit message: USB Port + DB Routed
Parts:
- moved F1 67.5 mm to (74.6, 47.6), turned to 180 degrees
- moved R3 51.9 mm to (53.2, 70.7)
- moved SW55 41.1 mm to (48.2, 69.6), turned to 180 degrees
- moved C1 1.15 mm to (65.1, 67.5)
- moved R2 0.90 mm to (158.2, 33.2)
- moved R1 0.73 mm to (153.5, 33.2)
Routing:
- net UD+: track 5.93 -> 107.1 mm, vias 0 -> 1
- net VCC: track 0.00 -> 98.9 mm, vias 0 -> 2
- net UD-: track 5.93 -> 104.0 mm, vias 0 -> 1
- net GND: track 11.8 -> 34.2 mm, vias 0 -> 3
- net Net-(SW12-Pad2): track 0.00 -> 19.1 mm
- net Net-(D6-Pad2): track 0.00 -> 16.9 mm
- net RESET: track 0.00 -> 12.0 mm
- net Net-(D1-Pad1): track 0.00 -> 11.2 mm
- net Net-(D6-Pad1): track 0.00 -> 11.2 mm
- net Net-(D5-Pad1): track 0.00 -> 11.2 mm
- net Net-(D4-Pad1): track 0.00 -> 11.2 mm
- net Net-(D2-Pad1): track 0.00 -> 11.2 mm
- net Net-(D3-Pad1): track 0.00 -> 11.2 mm
- net Net-(D3-Pad2): track 0.00 -> 7.34 mm
- net Net-(D2-Pad2): track 0.00 -> 7.34 mm
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- added copper zone on B.Cu, net GND
- added copper zone on F.Cu, net GND
Other:
- outline, holes or cut-outs redrawn
