File: pcb/QS-13u.kicad_pcb (KiCad board)
At the start: 2 copper layers, 247.6 x 84.9 mm, 100 parts, among them J1 Conn_01x04, J2 USB_C_Receptacle_USB2.0, SW1 MX_SW_solder, SW10 MX_SW_solder, SW11 MX_SW_solder, SW12 MX_SW_solder, SW13 MX_SW_solder, SW14 MX_SW_solder, SW15 MX_SW_solder, SW16 MX_SW_solder, SW17 MX_SW_solder, SW18 MX_SW_solder, SW19 MX_SW_solder, SW2 MX_SW_solder, SW20 MX_SW_solder, SW21 MX_SW_solder, SW22 MX_SW_solder, SW23 MX_SW_solder, SW24 MX_SW_solder, SW25 MX_SW_solder, SW26 MX_SW_solder, SW27 MX_SW_solder, SW28 MX_SW_solder, SW29 MX_SW_solder, SW3 MX_SW_solder, SW30 MX_SW_solder, SW31 MX_SW_solder, SW32 MX_SW_solder, SW33 MX_SW_solder, SW34 MX_SW_solder, SW35 MX_SW_solder, SW36 MX_SW_solder, SW37 MX_SW_solder, SW38 MX_SW_solder, SW39 MX_SW_solder, SW4 MX_SW_solder, SW40 MX_SW_solder, SW41 MX_SW_solder, SW42 MX_SW_solder, SW43 MX_SW_solder, SW44 MX_SW_solder, SW45 MX_SW_solder, SW46 MX_SW_solder, SW47 MX_SW_solder, SW48 MX_SW_solder, SW49 MX_SW_solder, SW5 MX_SW_solder, SW50 MX_SW_solder, SW51 MX_SW_solder, SW52 MX_SW_solder, SW53 MX_SW_solder, SW54 MX_SW_solder, SW55 SW_Push, SW6 MX_SW_solder, SW7 MX_SW_solder, SW8 MX_SW_solder, SW9 MX_SW_solder, U1 USBLC6-2SC6, U2 ATmega32U2-M, Y1 16 MHz

Commit message: PCB Rev.1
Everything seems to be connected and no obvious errors were found
Parts:
- R4, R5: value 10k -> 22
- moved D22 41.3 mm to (214.3, 100.8)
- moved D7 21.1 mm to (74.6, 62.7)
- moved D23 6.24 mm to (261.8, 88.9), turned to 90 degrees
- moved D18 1.12 mm to (258.0, 81.8)
- renumbered SW55 to RESET1
Connections:
- D1 pad 3: Net-(D1-Pad3) -> ROW3
- D10 pad 3: Net-(D10-Pad3) -> ROW2
- D11 pad 3: Net-(D10-Pad3) -> ROW2
- D12 pad 3: Net-(D10-Pad3) -> ROW2
- D13 pad 3: Net-(D13-Pad3) -> ROW1
- D14 pad 3: Net-(D13-Pad3) -> ROW1
- D15 pad 3: Net-(D13-Pad3) -> ROW1
- D16 pad 3: Net-(D13-Pad3) -> ROW1
- D17 pad 3: Net-(D13-Pad3) -> ROW1
- D18 pad 3: Net-(D13-Pad3) -> ROW1
- D19 pad 3: Net-(D19-Pad3) -> ROW0
- D2 pad 3: Net-(D1-Pad3) -> ROW3
- D20 pad 3: Net-(D19-Pad3) -> ROW0
- D21 pad 3: Net-(D19-Pad3) -> ROW0
- D22 pad 3: Net-(D19-Pad3) -> ROW0
- D23 pad 3: Net-(D19-Pad3) -> ROW0
- D3 pad 3: Net-(D1-Pad3) -> ROW3
- D4 pad 3: Net-(D1-Pad3) -> ROW3
- D5 pad 3: Net-(D1-Pad3) -> ROW3
- D6 pad 3: Net-(D1-Pad3) -> ROW3
- D7 pad 3: Net-(D10-Pad3) -> ROW2
- D8 pad 3: Net-(D10-Pad3) -> ROW2
- D9 pad 3: Net-(D10-Pad3) -> ROW2
- J2 pad S1: unconnected-(J2-PadS1) -> GND
- SW1 pad 1: Net-(SW1-Pad1) -> COL0
- SW10 pad 2: Net-(SW10-Pad2) -> COL9
- SW11 pad 1: Net-(SW11-Pad1) -> COL10
- SW12 pad 2: Net-(SW12-Pad2) -> COL11
- SW13 pad 2: Net-(SW12-Pad2) -> COL11
- SW14 pad 1: Net-(SW1-Pad1) -> COL0
- SW14 pad 2: Net-(D7-Pad1) -> Net-(D7-Pad2)
- SW15 pad 1: Net-(D7-Pad2) -> Net-(D7-Pad1)
- SW15 pad 2: Net-(SW15-Pad2) -> COL1
- SW16 pad 1: Net-(SW16-Pad1) -> COL2
- SW17 pad 2: Net-(SW17-Pad2) -> COL3
- SW18 pad 1: Net-(SW18-Pad1) -> COL4
- SW19 pad 2: Net-(SW19-Pad2) -> COL5
- SW2 pad 2: Net-(SW15-Pad2) -> COL1
- SW20 pad 1: Net-(SW20-Pad1) -> COL6
- SW21 pad 2: Net-(SW21-Pad2) -> COL7
- SW22 pad 1: Net-(SW22-Pad1) -> COL8
- SW23 pad 2: Net-(SW10-Pad2) -> COL9
- SW24 pad 1: Net-(SW11-Pad1) -> COL10
- SW25 pad 2: Net-(SW12-Pad2) -> COL11
- SW26 pad 1: Net-(SW1-Pad1) -> COL0
- SW27 pad 2: Net-(SW15-Pad2) -> COL1
- SW28 pad 1: Net-(SW16-Pad1) -> COL2
- SW29 pad 2: Net-(SW17-Pad2) -> COL3
- SW3 pad 1: Net-(SW16-Pad1) -> COL2
- SW30 pad 1: Net-(SW18-Pad1) -> COL4
- SW31 pad 2: Net-(SW19-Pad2) -> COL5
- SW32 pad 1: Net-(SW20-Pad1) -> COL6
- SW33 pad 2: Net-(SW21-Pad2) -> COL7
- SW34 pad 1: Net-(SW22-Pad1) -> COL8
- SW35 pad 2: Net-(SW10-Pad2) -> COL9
- SW36 pad 1: Net-(SW11-Pad1) -> COL10
- SW37 pad 2: Net-(SW12-Pad2) -> COL11
- SW38 pad 1: Net-(SW11-Pad1) -> COL10
- SW39 pad 1: Net-(SW1-Pad1) -> COL0
- SW4 pad 2: Net-(SW17-Pad2) -> COL3
- SW40 pad 2: Net-(SW15-Pad2) -> COL1
- SW41 pad 1: Net-(SW16-Pad1) -> COL2
- SW42 pad 1: Net-(SW18-Pad1) -> COL4
- SW43 pad 2: Net-(SW19-Pad2) -> COL5
- SW44 pad 1: Net-(SW22-Pad1) -> COL8
- SW45 pad 2: Net-(SW10-Pad2) -> COL9
- SW46 pad 1: Net-(SW11-Pad1) -> COL10
- SW47 pad 2: Net-(SW12-Pad2) -> COL11
- SW48 pad 1: Net-(SW1-Pad1) -> COL0
- SW49 pad 1: Net-(SW16-Pad1) -> COL2
- SW5 pad 1: Net-(SW18-Pad1) -> COL4
- SW50 pad 1: Net-(SW18-Pad1) -> COL4
- SW51 pad 2: Net-(SW19-Pad2) -> COL5
- SW52 pad 1: Net-(SW22-Pad1) -> COL8
- SW53 pad 1: Net-(SW11-Pad1) -> COL10
- SW54 pad 2: Net-(SW12-Pad2) -> COL11
- SW6 pad 2: Net-(SW19-Pad2) -> COL5
- SW7 pad 1: Net-(SW20-Pad1) -> COL6
- SW8 pad 2: Net-(SW21-Pad2) -> COL7
- SW9 pad 1: Net-(SW22-Pad1) -> COL8
- U2 pad 10: unconnected-(U2-Pad10) -> COL7
- U2 pad 11: unconnected-(U2-Pad11) -> COL6
- U2 pad 12: unconnected-(U2-Pad12) -> COL3
- U2 pad 14: unconnected-(U2-Pad14) -> ROW1
- U2 pad 15: unconnected-(U2-Pad15) -> COL8
- U2 pad 16: unconnected-(U2-Pad16) -> COL5
- U2 pad 17: unconnected-(U2-Pad17) -> COL4
- U2 pad 18: unconnected-(U2-Pad18) -> COL2
- U2 pad 19: unconnected-(U2-Pad19) -> COL1
- U2 pad 20: unconnected-(U2-Pad20) -> ROW0
- U2 pad 23: unconnected-(U2-Pad23) -> COL0
- U2 pad 25: unconnected-(U2-Pad25) -> ROW3
- U2 pad 6: unconnected-(U2-Pad6) -> ROW2
- U2 pad 7: unconnected-(U2-Pad7) -> COL11
- U2 pad 8: unconnected-(U2-Pad8) -> COL10
- U2 pad 9: unconnected-(U2-Pad9) -> COL9
Routing:
- net COL8: track 0.00 -> 282.4 mm
- net COL11: track 0.00 -> 276.4 mm
- net COL10: track 0.00 -> 276.1 mm
- net ROW0: track 0.00 -> 250.2 mm
- net COL9: track 0.00 -> 247.3 mm
- net ROW3: track 0.00 -> 225.1 mm, vias 0 -> 4
- net COL5: track 0.00 -> 215.7 mm
- net ROW1: track 0.00 -> 206.6 mm
- net ROW2: track 0.00 -> 190.8 mm
- net COL7: track 0.00 -> 181.0 mm
- net COL4: track 0.00 -> 174.1 mm
- net COL6: track 0.00 -> 158.1 mm
- net COL2: track 0.00 -> 114.7 mm
- net COL3: track 0.00 -> 105.2 mm
- net COL1: track 0.00 -> 101.2 mm
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Other:
- outline, holes or cut-outs redrawn

Commit message: Added art and adjusted gerbers
Parts:
- added Ref**: Val**, extra:thinking, B.Cu at (197.5, 97.4)
- added Ref**: Val**, qw new logo:qw-logo-small, B.Cu at (36.3, 52.4)
Other:
- board text added: "Dude literally that whole server is toxic. You guys just pretend everything is fine. if anyone gives their opinions or tries to have serious discussions they just put emotes and start making fun of each other."
- board text added: "QS-13u PCB by Quark With love for my favourite 40% degens, Solar and Afmuente quark.works"

Commit message: Afmuente -> Muente
Other:
- board text added: "QS-13u PCB by Quark With love for my favourite 40% degens, Solar and Muente quark.works"
- board text removed: "QS-13u PCB by Quark With love for my favourite 40% degens, Solar and Afmuente quark.works"
